File: V4.0/AUX power board (V4.0).sch (EAGLE design)
At the start: 51 parts, among them U1 ATMEGA328P_TQFP

Commit message: Add current sensor
Still need new 5V regulator and a -12V source for the op amps
Parts:
- added R4: 1k, resistor:R-US_R0603
- added U$1: ACS723, linear:ACS723
- added VOLTAGE_BUFFER2: OPA340N, burr-brown:OPA340N
- C5: value 2.2uF -> 0.1uF
Connections:
- net N$11 renamed BATTERY_V(0-5)
- removed net MEASUREMENT_OUT: C5.1, C6.1, POWERHEADER.1, U1.PC0(ADC0)
- new net I_MEASUREMENT_OUT: C5.1, C6.1, POWERHEADER.1, U1.PC0(ADC0), VOLTAGE_BUFFER2.-IN, VOLTAGE_BUFFER2.OUT
- new net N$2: U$1.P$7, VOLTAGE_BUFFER2.+IN
- new net N$3: R10.2, R4.1
- net FUSED_BATTERY_IN+: now also U$1.P$1, U$1.P$2
- net GND: now also U$1.P$5, U$1.P$6; no longer VOLTAGE_BUFFER1.V-
- net INPUT_UNREG: now also U$1.P$3, U$1.P$4
- net OUTPUT_12REG: now also R4.2; no longer R10.2
- net OUTPUT_5REG: now also U$1.P$8
Other:
- note added: "-12V for OPAMPS"
- note added: "C15 see ~1.7A ripple"
- note added: "This needs to be replaced. I want to get rid of electrolytics"
- note removed: "+/-15V for OPAMPs"
- note removed: "Ensure to include power loss of ALL components on this board!"
- moved on the sheet: C5, C6, C9, R3, R6, VOLTAGE_BUFFER1
