File: V4.0 In Development/AUX power board (V4.0).sch (EAGLE design)
At the start: 89 parts, among them U1 ATMEGA328P_TQFP, U2 TPS5405DR, U3 LTC4365HTS8TRMPBFTSOT-23_TS8-M

Commit message: Minor Changes/tweaks
Parts:
- removed 1M1: 1820k, rcl:R-US_R0805
Connections:
- net N$19: no longer R18.1
- net N$28: no longer 1M1.1
- net NEG_TERMINAL: now also R18.1; no longer 1M1.2
Other:
- note added: "Overvoltage Protection PSMN1R4-40YLDX nMOS"
- note added: "Reverse Polarity Protection PSMN1R4-40YLDX nMOS"
- note added: "Reverse polarity indicator"
- note removed: "Reverse Polarity Protection. PSMN1R4-40YLDX nMOS"
Changed lines of the file:
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@@
 <part name="GND11" library="supply1" deviceset="GND" device=""/>
 <part name="1M" library="rcl" deviceset="R-US_" device="R0805" value="1820k"/>
-<part name="1M1" library="rcl" deviceset="R-US_" device="R0805" value="1820k"/>
 </parts>
 <sheets>
@@
 10uH per coil</text>
 <text x="160.782" y="156.718" size="1.27" layer="91">10uH</text>
-<text x="93.98" y="30.48" size="1.778" layer="91">Reverse Polarity Protection.
+<text x="101.6" y="25.4" size="1.778" layer="91">Overvoltage Protection
 PSMN1R4-40YLDX nMOS</text>
 <text x="43.18" y="0" size="1.778" layer="91">blown fuse ind.</text>
+<text x="66.04" y="27.94" size="1.778" layer="91">Reverse polarity
+indicator</text>
+<text x="66.04" y="-25.4" size="1.778" layer="91">Reverse Polarity Protection
+PSMN1R4-40YLDX nMOS</text>
 </plain>
 <instances>
@@
 <instance part="GND11" gate="1" x="91.44" y="-12.7"/>
 <instance part="1M" gate="G$1" x="86.36" y="-2.54" rot="R270"/>
-<instance part="1M1" gate="G$1" x="33.02" y="7.62" rot="R270"/>
 </instances>
 <busses>
@@
 <wire x1="27.94" y1="-2.54" x2="30.48" y2="-2.54" width="0.1524" layer="91"/>
 <wire x1="30.48" y1="-2.54" x2="30.48" y2="-10.16" width="0.1524" layer="91"/>
-<wire x1="30.48" y1="-10.16" x2="38.1" y2="-10.16" width="0.1524" layer="91"/>
 <pinref part="LED1" gate="G$1" pin="C"/>
-<wire x1="38.1" y1="-10.16" x2="63.5" y2="-10.16" width="0.1524" layer="91"/>
+<wire x1="30.48" y1="-10.16" x2="63.5" y2="-10.16" width="0.1524" layer="91"/>
 <wire x1="63.5" y1="-5.08" x2="63.5" y2="-10.16" width="0.1524" layer="91"/>
 <junction x="63.5" y="-10.16"/>
@@
 <pinref part="PSMN1R4-40TLDX1" gate="G$1" pin="D"/>
 <wire x1="63.5" y1="-10.16" x2="71.12" y2="-12.7" width="0.1524" layer="91"/>
-<pinref part="1M1" gate="G$1" pin="2"/>
-<wire x1="33.02" y1="2.54" x2="38.1" y2="-10.16" width="0.1524" layer="91"/>
-<junction x="38.1" y="-10.16"/>
+<pinref part="R18" gate="G$1" pin="1"/>
+<wire x1="73.66" y1="-2.54" x2="73.66" y2="-5.08" width="0.1524" layer="91"/>
+<wire x1="63.5" y1="-10.16" x2="68.58" y2="-10.16" width="0.1524" layer="91"/>
+<wire x1="68.58" y1="-10.16" x2="73.66" y2="-5.08" width="0.1524" layer="91"/>
 </segment>
 </net>
@@
 <wire x1="86.36" y1="5.08" x2="86.36" y2="2.54" width="0.1524" layer="91"/>
 <junction x="86.36" y="5.08"/>
-<pinref part="1M1" gate="G$1" pin="1"/>
-<wire x1="33.02" y1="12.7" x2="45.72" y2="12.7" width="0.1524" layer="91"/>
-<junction x="45.72" y="12.7"/>
 </segment>
 </net>
@@
 <wire x1="78.74" y1="2.54" x2="81.28" y2="2.54" width="0.1524" layer="91"/>
 <pinref part="R20" gate="G$1" pin="1"/>
-<pinref part="R18" gate="G$1" pin="1"/>
-<wire x1="73.66" y1="-2.54" x2="73.66" y2="-5.08" width="0.1524" layer="91"/>
-<wire x1="73.66" y1="-5.08" x2="76.2" y2="-5.08" width="0.1524" layer="91"/>
 <junction x="76.2" y="-5.08"/>
 <pinref part="TN2540-600G-TR" gate="G$1" pin="C"/>

Commit message: Added Jumpers to enable/disable data-logging
cheap solution to avoid wasting power
Parts:
- added JP1, JP2: (no value), SparkFun (2015_10_14 22_27_04 UTC):M03PTH
Connections:
- new net DATA_LOG_POWER_12V: C22.1, GMK107BJ104KAHT1.1, JP1.2, U$8.V+, VOLTAGE_BUFFER1.V+
- new net DATA_LOG_POWER_5V: C2.1, C26.1, JP2.2, MLZ2012DR10DT000.1, MURS120T3G1.C, R14.2, U$1.P$8, U1.VCC@4, U1.VCC@6
- net GND: now also JP1.3, JP2.3
- net OUTPUT_12REG: now also JP1.1; no longer C22.1, GMK107BJ104KAHT1.1, U$8.V+, VOLTAGE_BUFFER1.V+
- net OUTPUT_5REG: now also JP2.1; no longer C2.1, C26.1, MLZ2012DR10DT000.1, MURS120T3G1.C, R14.2, U$1.P$8, U1.VCC@4, U1.VCC@6
Changed lines of the file:
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@@
 <part name="GND11" library="supply1" deviceset="GND" device=""/>
 <part name="1M" library="rcl" deviceset="R-US_" device="R0805" value="1820k"/>
+<part name="JP1" library="SparkFun (2015_10_14 22_27_04 UTC)" deviceset="M03" device="PTH"/>
+<part name="JP2" library="SparkFun (2015_10_14 22_27_04 UTC)" deviceset="M03" device="PTH"/>
+<part name="GND35" library="E-P-008-R1.2" deviceset="GND" device=""/>
+<part name="GND36" library="E-P-008-R1.2" deviceset="GND" device=""/>
 </parts>
 <sheets>
@@
 <instance part="GND11" gate="1" x="91.44" y="-12.7"/>
 <instance part="1M" gate="G$1" x="86.36" y="-2.54" rot="R270"/>
+<instance part="JP1" gate="G$1" x="317.5" y="33.02" rot="R90"/>
+<instance part="JP2" gate="G$1" x="302.26" y="33.02" rot="R90"/>
+<instance part="GND35" gate="1" x="292.1" y="38.1"/>
+<instance part="GND36" gate="1" x="309.88" y="38.1"/>
 </instances>
 <busses>
@@
 </segment>
 <segment>
-<pinref part="VOLTAGE_BUFFER1" gate="G$1" pin="V+"/>
-<wire x1="154.94" y1="73.66" x2="154.94" y2="68.58" width="0.1524" layer="91"/>
-<label x="154.94" y="73.66" size="1.27" layer="95" rot="MR270"/>
-<wire x1="154.94" y1="73.66" x2="154.94" y2="68.58" width="0.1524" layer="91"/>
-</segment>
-<segment>
 <pinref part="C11" gate="G$1" pin="1"/>
 <wire x1="144.78" y1="231.14" x2="147.32" y2="231.14" width="0.1524" layer="91"/>
@@
 </segment>
 <segment>
-<wire x1="73.66" y1="66.04" x2="73.66" y2="60.96" width="0.1524" layer="91"/>
-<label x="73.66" y="60.96" size="1.778" layer="95"/>
-</segment>
-<segment>
-<pinref part="U$8" gate="G$1" pin="V+"/>
-<wire x1="312.42" y1="93.98" x2="335.28" y2="93.98" width="0.1524" layer="91"/>
-<pinref part="GMK107BJ104KAHT1" gate="G$1" pin="1"/>
-<wire x1="335.28" y1="93.98" x2="350.52" y2="93.98" width="0.1524" layer="91"/>
-<junction x="335.28" y="93.98"/>
-<pinref part="C22" gate="G$1" pin="1"/>
-<label x="350.52" y="93.98" size="1.778" layer="95" rot="R90"/>
+<pinref part="JP1" gate="G$1" pin="1"/>
+<wire x1="320.04" y1="43.18" x2="320.04" y2="40.64" width="0.1524" layer="91"/>
+<label x="320.04" y="43.18" size="1.778" layer="95"/>
 </segment>
 </net>
@@
 <junction x="86.36" y="-10.16"/>
 </segment>
+<segment>
+<pinref part="JP2" gate="G$1" pin="3"/>
+<wire x1="299.72" y1="40.64" x2="299.72" y2="43.18" width="0.1524" layer="91"/>
+<wire x1="299.72" y1="43.18" x2="292.1" y2="43.18" width="0.1524" layer="91"/>
+<wire x1="292.1" y1="43.18" x2="292.1" y2="40.64" width="0.1524" layer="91"/>
+<pinref part="GND35" gate="1" pin="GND"/>
+</segment>
+<segment>
+<pinref part="JP1" gate="G$1" pin="3"/>
+<wire x1="314.96" y1="40.64" x2="314.96" y2="43.18" width="0.1524" layer="91"/>
+<wire x1="314.96" y1="43.18" x2="309.88" y2="43.18" width="0.1524" layer="91"/>
+<wire x1="309.88" y1="43.18" x2="309.88" y2="40.64" width="0.1524" layer="91"/>
+<pinref part="GND36" gate="1" pin="GND"/>
+</segment>
 </net>
 <net name="OUTPUT_5REG" class="0">
-<segment>
-<wire x1="261.62" y1="182.88" x2="236.22" y2="182.88" width="0.1524" layer="91"/>
-<wire x1="236.22" y1="182.88" x2="236.22" y2="180.34" width="0.1524" layer="91"/>
-<junction x="236.22" y="182.88"/>
-<pinref part="C2" gate="G$1" pin="1"/>
-<label x="205.74" y="182.88" size="1.778" layer="95"/>
-<wire x1="223.52" y1="182.88" x2="226.06" y2="182.88" width="0.1524" layer="91"/>
-<wire x1="226.06" y1="182.88" x2="236.22" y2="182.88" width="0.1524" layer="91"/>
-<wire x1="236.22" y1="182.88" x2="236.22" y2="187.96" width="0.1524" layer="91"/>
-<pinref part="MLZ2012DR10DT000" gate="G$1" pin="1"/>
-<pinref part="U1" gate="U$1" pin="VCC@4"/>
-<pinref part="U1" gate="U$1" pin="VCC@6"/>
-<wire x1="261.62" y1="182.88" x2="261.62" y2="180.34" width="0.1524" layer="91"/>
-<junction x="261.62" y="182.88"/>
-<wire x1="226.06" y1="180.34" x2="226.06" y2="182.88" width="0.1524" layer="91"/>
-<junction x="226.06" y="182.88"/>
-<pinref part="C26" gate="G$1" pin="1"/>
-</segment>
-<segment>
-<wire x1="236.22" y1="203.2" x2="236.22" y2="213.36" width="0.1524" layer="91"/>
-<wire x1="236.22" y1="213.36" x2="241.3" y2="213.36" width="0.1524" layer="91"/>
-<pinref part="MURS120T3G1" gate="G$1" pin="C"/>
-<wire x1="241.3" y1="213.36" x2="246.38" y2="213.36" width="0.1524" layer="91"/>
-<wire x1="246.38" y1="213.36" x2="246.38" y2="200.66" width="0.1524" layer="91"/>
-<wire x1="241.3" y1="213.36" x2="241.3" y2="215.9" width="0.1524" layer="91"/>
-<junction x="241.3" y="213.36"/>
-<label x="241.3" y="215.9" size="1.778" layer="95"/>
-<pinref part="R14" gate="G$1" pin="2"/>
-</segment>
 <segment>
 <wire x1="340.36" y1="-10.16" x2="345.44" y2="-10.16" width="0.1524" layer="91"/>
@@
 </segment>
 <segment>
-<pinref part="U$1" gate="G$1" pin="P$8"/>
-<wire x1="50.8" y1="81.28" x2="60.96" y2="81.28" width="0.1524" layer="91"/>
-<label x="60.96" y="81.28" size="1.778" layer="95" rot="R90"/>
-</segment>
-<segment>
 <pinref part="SV1" gate="1" pin="3"/>
 <wire x1="342.9" y1="33.02" x2="342.9" y2="35.56" width="0.1524" layer="91"/>
@@
 <pinref part="R2" gate="G$1" pin="2"/>
 <pinref part="R5" gate="G$1" pin="2"/>
+</segment>
+<segment>
+<label x="304.8" y="43.18" size="1.778" layer="95" rot="R90"/>
+<pinref part="JP2" gate="G$1" pin="1"/>
+<wire x1="304.8" y1="43.18" x2="304.8" y2="40.64" width="0.1524" layer="91"/>
 </segment>
 </net>
@@
 </segment>
 </net>
+<net name="DATA_LOG_POWER_5V" class="0">
+<segment>
+<label x="274.32" y="48.26" size="1.778" layer="95"/>
+<pinref part="JP2" gate="G$1" pin="2"/>
+<wire x1="302.26" y1="40.64" x2="302.26" y2="48.26" width="0.1524" layer="91"/>
+<wire x1="302.26" y1="48.26" x2="299.72" y2="48.26" width="0.1524" layer="91"/>
+</segment>
+<segment>
+<pinref part="U$1" gate="G$1" pin="P$8"/>
+<wire x1="50.8" y1="81.28" x2="60.96" y2="81.28" width="0.1524" layer="91"/>
+<label x="60.96" y="81.28" size="1.778" layer="95" rot="R90"/>
+</segment>
+<segment>
+<wire x1="261.62" y1="182.88" x2="236.22" y2="182.88" width="0.1524" layer="91"/>
+<wire x1="236.22" y1="182.88" x2="236.22" y2="180.34" width="0.1524" layer="91"/>
+<junction x="236.22" y="182.88"/>
+<pinref part="C2" gate="G$1" pin="1"/>
+<label x="200.66" y="182.88" size="1.778" layer="95"/>
+<wire x1="223.52" y1="182.88" x2="226.06" y2="182.88" width="0.1524" layer="91"/>
+<wire x1="226.06" y1="182.88" x2="236.22" y2="182.88" width="0.1524" layer="91"/>
+<wire x1="236.22" y1="182.88" x2="236.22" y2="187.96" width="0.1524" layer="91"/>
+<pinref part="MLZ2012DR10DT000" gate="G$1" pin="1"/>
+<pinref part="U1" gate="U$1" pin="VCC@4"/>
+<pinref part="U1" gate="U$1" pin="VCC@6"/>
+<wire x1="261.62" y1="182.88" x2="261.62" y2="180.34" width="0.1524" layer="91"/>
+<junction x="261.62" y="182.88"/>
+<wire x1="226.06" y1="180.34" x2="226.06" y2="182.88" width="0.1524" layer="91"/>
+<junction x="226.06" y="182.88"/>
+<pinref part="C26" gate="G$1" pin="1"/>
+</segment>
+<segment>
+<wire x1="236.22" y1="203.2" x2="236.22" y2="213.36" width="0.1524" layer="91"/>
+<wire x1="236.22" y1="213.36" x2="241.3" y2="213.36" width="0.1524" layer="91"/>
+<pinref part="MURS120T3G1" gate="G$1" pin="C"/>
+<wire x1="241.3" y1="213.36" x2="246.38" y2="213.36" width="0.1524" layer="91"/>
+<wire x1="246.38" y1="213.36" x2="246.38" y2="200.66" width="0.1524" layer="91"/>
+<wire x1="241.3" y1="213.36" x2="241.3" y2="215.9" width="0.1524" layer="91"/>
+<junction x="241.3" y="213.36"/>
+<label x="241.3" y="215.9" size="1.778" layer="95"/>
+<pinref part="R14" gate="G$1" pin="2"/>
+</segment>
+</net>
+<net name="DATA_LOG_POWER_12V" class="0">
+<segment>
+<label x="317.5" y="43.18" size="1.778" layer="95" rot="R90"/>
+<pinref part="JP1" gate="G$1" pin="2"/>
+<wire x1="314.96" y1="45.72" x2="317.5" y2="45.72" width="0.1524" layer="91"/>
+<wire x1="317.5" y1="45.72" x2="317.5" y2="40.64" width="0.1524" layer="91"/>
+</segment>
+<segment>
+<pinref part="U$8" gate="G$1" pin="V+"/>
+<wire x1="312.42" y1="93.98" x2="335.28" y2="93.98" width="0.1524" layer="91"/>
+<pinref part="GMK107BJ104KAHT1" gate="G$1" pin="1"/>
+<wire x1="335.28" y1="93.98" x2="350.52" y2="93.98" width="0.1524" layer="91"/>
+<junction x="335.28" y="93.98"/>
+<pinref part="C22" gate="G$1" pin="1"/>
+<label x="350.52" y="93.98" size="1.778" layer="95" rot="R90"/>
+</segment>
+<segment>
+<pinref part="VOLTAGE_BUFFER1" gate="G$1" pin="V+"/>
+<wire x1="154.94" y1="73.66" x2="154.94" y2="68.58" width="0.1524" layer="91"/>
+<label x="154.94" y="73.66" size="1.27" layer="95" rot="MR270"/>
+<wire x1="154.94" y1="73.66" x2="154.94" y2="68.58" width="0.1524" layer="91"/>
+</segment>
+<segment>
+<wire x1="73.66" y1="66.04" x2="73.66" y2="60.96" width="0.1524" layer="91"/>
+<label x="73.66" y="60.96" size="1.778" layer="95"/>
+</segment>
+</net>
