File: V4.0 In Development/AUX power board (V4.0).sch (EAGLE design)
At the start: 95 parts, among them U1 ATMEGA328P_TQFP, U2 TPS5405DR

Commit message: Accidently saved as EAGLE 8.2
EAGLE 8.2+ changed how it saves projects. I had to re-save for legacy
support (I believe our members are using version 7.x)
Parts:
- R20, R4: device resistor:R-US_0817/22 -> resistor@1:R-US_0817/22
Changed lines of the file:
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@@
 <part name="1N5356BRLG_1" library="diode" deviceset="ZENER-DIODE" device="DO41Z10" value="19V"/>
 <part name="LED2" library="E-P-008-R1.2" deviceset="LED" device="SML1206" value="RED"/>
-<part name="R20" library="resistor" library_urn="urn:adsk.eagle:library:348" deviceset="R-US_" device="0817/22" value="400 (5W)"/>
+<part name="R20" library="resistor@1" deviceset="R-US_" device="0817/22" value="400 (5W)"/>
 <part name="GND11" library="supply1" deviceset="GND" device=""/>
 <part name="R10" library="rcl" deviceset="R-US_" device="R0805" value="1M"/>
@@
 <part name="AL5809-20S1-7_5" library="semicon-smd-ipc" deviceset="D-" device="SOD123" value="20mA"/>
 <part name="C35" library="rcl" deviceset="C-EU" device="C1210" value="22uF"/>
-<part name="R4" library="resistor" library_urn="urn:adsk.eagle:library:348" deviceset="R-US_" device="0817/22" value="400 (5W)"/>
+<part name="R4" library="resistor@1" deviceset="R-US_" device="0817/22" value="400 (5W)"/>
 <part name="PSMN1R4-40YLDX2" library="PSMN1R4-40YLDX" deviceset="MOSFET-NCHANNEL" device="FDS6630A"/>
 <part name="LED3" library="E-P-008-R1.2" deviceset="LED" device="SML1206" value="RED"/>
@@
 which will not be processed correctly with this version.
 </note>
-<note version="8.2" severity="warning">
-Since Version 8.2, Eagle supports online libraries. The ids
-of those online libraries will not be understood (or retained)
-with this version.
-</note>
 </compatibility>

Commit message: Changed Crowbar
The top of the zener is attached before the fuse. That way if the SCR is
triggered due to over voltage, the fault LEDs will stay illuminated.
Connections:
- net BATTERY_IN_UNFUSED+: now also 1N5354BRLG.C
- net INPUT_UNREG: no longer 1N5354BRLG.C
Changed lines of the file:
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@@
 <?xml version="1.0" encoding="utf-8"?>
 <!DOCTYPE eagle SYSTEM "eagle.dtd">
-<eagle version="8.2.1">
+<eagle version="7.5.0">
 <drawing>
 <settings>
@@
 <wire x1="63.5" y1="20.32" x2="73.66" y2="20.32" width="0.1524" layer="91"/>
 <wire x1="73.66" y1="20.32" x2="81.28" y2="20.32" width="0.1524" layer="91"/>
-<wire x1="81.28" y1="20.32" x2="86.36" y2="20.32" width="0.1524" layer="91"/>
-<wire x1="86.36" y1="20.32" x2="129.54" y2="20.32" width="0.1524" layer="91"/>
+<wire x1="81.28" y1="20.32" x2="129.54" y2="20.32" width="0.1524" layer="91"/>
 <wire x1="104.14" y1="20.32" x2="129.54" y2="20.32" width="0.1524" layer="91"/>
 <pinref part="R20" gate="G$1" pin="2"/>
@@
 <wire x1="81.28" y1="10.16" x2="81.28" y2="20.32" width="0.1524" layer="91"/>
 <junction x="81.28" y="20.32"/>
-<wire x1="86.36" y1="20.32" x2="86.36" y2="17.78" width="0.1524" layer="91"/>
-<junction x="86.36" y="20.32"/>
-<pinref part="1N5354BRLG" gate="G$1" pin="C"/>
 <pinref part="BT152B-400R" gate="G$1" pin="D"/>
 <wire x1="129.54" y1="10.16" x2="129.54" y2="20.32" width="0.1524" layer="91"/>
@@
 <wire x1="38.1" y1="7.62" x2="43.18" y2="7.62" width="0.1524" layer="91"/>
 <pinref part="FUSE" gate="G$1" pin="1"/>
-<wire x1="38.1" y1="20.32" x2="53.34" y2="20.32" width="0.1524" layer="91"/>
+<wire x1="38.1" y1="20.32" x2="50.8" y2="20.32" width="0.1524" layer="91"/>
+<wire x1="50.8" y1="20.32" x2="53.34" y2="20.32" width="0.1524" layer="91"/>
+<wire x1="50.8" y1="20.32" x2="50.8" y2="30.48" width="0.1524" layer="91"/>
+<junction x="50.8" y="20.32"/>
+<wire x1="50.8" y1="30.48" x2="88.9" y2="30.48" width="0.1524" layer="91"/>
+<wire x1="88.9" y1="30.48" x2="88.9" y2="22.86" width="0.1524" layer="91"/>
+<pinref part="1N5354BRLG" gate="G$1" pin="C"/>
+<wire x1="88.9" y1="22.86" x2="86.36" y2="22.86" width="0.1524" layer="91"/>
+<wire x1="86.36" y1="22.86" x2="86.36" y2="17.78" width="0.1524" layer="91"/>
 </segment>
 </net>

Commit message: Trying this commit again
Parts:
- removed EEE-FP1V221AP3, EEE-FP1V221AP4: 220uF, rcl:CPOL-US175TMP-0808
- added C24, C25: UPJ1V220MDD1TD, UPJ1V220MDD1TD:UPJ1V220MDD1TD
Connections:
- net BATTERY_IN_UNFUSED+: no longer 1N5354BRLG.C
- net DATA_LOG_POWER_5V: now also C7.1
- net GND: now also C25.11, C3.2; no longer EEE-FP1V221AP3.-, EEE-FP1V221AP4.-
- net INPUT_UNREG: now also 1N5354BRLG.C; no longer C7.1
- net N$11: now also C24.22; no longer C3.2
- net N$16: now also C24.11; no longer C3.1
- net N$26: no longer EEE-FP1V221AP4.+
- net OUTPUT_12NEG: now also C25.22; no longer C11.1
- net OUTPUT_12REG: now also C11.1, C3.1; no longer EEE-FP1V221AP3.+
Other:
- moved on the sheet: C11, C3, C30, C31, C7

Commit message: when git fails to sync
Parts:
- removed C24, C25: UPJ1V220MDD1TD, UPJ1V220MDD1TD:UPJ1V220MDD1TD
- added EEE-FP1V221AP3, EEE-FP1V221AP4: 220uF, rcl:CPOL-US175TMP-0808
Connections:
- net BATTERY_IN_UNFUSED+: now also 1N5354BRLG.C
- net DATA_LOG_POWER_5V: no longer C7.1
- net GND: now also EEE-FP1V221AP3.-, EEE-FP1V221AP4.-; no longer C25.11, C3.2
- net INPUT_UNREG: now also C7.1; no longer 1N5354BRLG.C
- net N$11: now also C3.2; no longer C24.22
- net N$16: now also C3.1; no longer C24.11
- net N$26: now also EEE-FP1V221AP4.+
- net OUTPUT_12NEG: now also C11.1; no longer C25.22
- net OUTPUT_12REG: now also EEE-FP1V221AP3.+; no longer C11.1, C3.1
Other:
- moved on the sheet: C11, C3, C30, C31, C7
