File: Milled Version/Aux_Power_Board.brd (EAGLE design)
At the start: 100 x 100 mm, 71 parts

Commit message: Made changes to aux power board, created horn board
Parts:
- removed C3: 10uF, SparkFun-Capacitors:0805
- removed C4, C5, C6: 0.1uF, SparkFun-Capacitors:0805
- removed CR1, CR2: MUR420RLG, MUR420RLG - Diode:DO-201AD
- removed FRAME3, FRAME4: FRAME-LEDGER, SparkFun-Aesthetics:CREATIVE_COMMONS
- removed JP3: (no value), jumper:JP1
- removed LED4, LED5, LED6, LED7: (no value), led:CHIP-LED0805
- removed R10, R11, R12, R13: (no value), rcl:M0805
- removed R4: 100k, SparkFun-Resistors:0805
- removed R5, R8, R9: 8.1MEG, SparkFun-Resistors:0805
- removed R6: 66.67k, SparkFun-Resistors:0805
- removed R7: 233.33k, SparkFun-Resistors:0805
- removed START.RELAY1: VCF4-1000, VCF4-1000:VCF4-1000
- removed U$11: CAP-8MM3.5MM, Eagle Library:CAP-8MM*3.5MM
- removed U$16, U$20: FUSEMINI-BLADE, Shell2013:MINI-BLADE-FUSE
- removed U$17, U$18, U$21, U$26, U$27: TE770966, Shell2013(1):2X1-MATE-N-LOCK
- removed U$19: 5W_RESISTOR, Eagle Library:5W_RESISTOR
- removed U$22, U$24: CAPESK108M025AH4EA, Shell2015:ESK108M025AH4EA
- removed U$23: LM2576, Shell2015:D2PAK-5
- removed U$25: M1418-ND, Shell2015:M1418-ND
- removed U$5: LT4365, Eagle Library:TSOT-23_TS8
- removed U$6: SI4946, Eagle Library:SOIC127P600X175-8N
- C1, C2: value 0.1uF -> (none); device SparkFun-Capacitors:0805 -> E-P-099-R2.2:0805
- U$8: value MBR360GOS -> CAPESK107M025AC3AA; device Shell2013:MBR360GOS -> Shell2015:ESK107M025AC3AA
- moved U$8 340.7 mm to (17.8, 5.08), turned to 180 degrees
- moved C2 308.4 mm to (65.4, 24.1), turned to 90 degrees
- moved C1 280.0 mm to (68.6, 24.1), turned to 90 degrees
- moved R2 123.9 mm to (53.3, 7.62)
- moved U$4 111.4 mm to (48.3, 22.9)
- moved U$9 104.5 mm to (49.5, 64.8)
- moved LED2 91.7 mm to (48.3, 7.62)
- moved LED1 78.9 mm to (59.7, 69.8)
- moved AUX_PWR1 70.1 mm to (66.0, 15.2), turned to 0 degrees
- moved AUX_PWR 69.6 mm to (85.1, 62.2), turned to 90 degrees
- moved U$3 69.5 mm to (71.1, 82.5)
- moved R3 62.2 mm to (63.5, 71.1)
- moved AUX_PWR2 62.1 mm to (85.1, 43.2), turned to 90 degrees
- moved AUX_PWR3 61.1 mm to (85.1, 24.1), turned to 90 degrees
- moved JP1 50.1 mm to (22.9, 35.6)
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Connections:
- net VIN_UNFUSED renamed VIN_
- removed net BATTERY_GND: C3.2, C4.2, C5.2, JP1.1, R1.1, R7.1, START.RELAY1.30, U$11.P$2, U$12.P$2, U$14.CIRCUIT2, U$15.CIRCUIT2, U$21.CIRCUIT2, U$5.4
- removed net FAULT': R10.1, U$5.6
- removed net GATE: U$5.8, U$6.2, U$6.4
- removed net N$10: CR2.2, U$18.CIRCUIT1, U$19.P$2
- removed net N$11: CR1.2, R11.1, START.RELAY1.85, U$17.CIRCUIT1
- removed net N$12: R13.2, START.RELAY1.87, U$19.P$1
- removed net N$13: JP3.1, R4.2
- removed net N$14: U$20.IN, U$21.CIRCUIT1
- removed net N$15: U$23.2, U$25.P$1, U$8.P$1
- removed net N$16: R8.2, R9.1, U$23.4
- removed net N$17: LED4.C, R10.2
- removed net N$18: LED5.C, R11.2
- removed net N$19: LED6.C, R12.2
- removed net N$2: R4.1, U$5.5
- removed net N$20: LED7.C, R13.1
- removed net N$4: R5.1, R6.2, U$5.2
- removed net N$5: R6.1, R7.2, U$5.3
- removed net N$8: CR2.1, LED7.A, U$16.OUT, U$18.CIRCUIT2
- removed net SERVO_POWER: C2.1, LED6.A, R9.2, U$24.P$1, U$25.P$2, U$26.CIRCUIT1
- removed net SOURCE1: U$6.1, U$6.3
- removed net VIN_FUSED: C3.1, C4.1, JP3.2, LED4.A, R5.2, U$13.OUT, U$5.1, U$6.7, U$6.8
- removed net VIN_PROTECTED: C5.1, JP2.2, U$11.P$1, U$12.P$1, U$16.IN, U$20.OUT, U$5.7, U$6.5, U$6.6
- new net GNDIN: JP1.1, R1.1, U$12.P$2, U$14.CIRCUIT2, U$15.CIRCUIT2
- net 12V: now also AUX_PWR.3, AUX_PWR.4, AUX_PWR1.3, AUX_PWR1.4, AUX_PWR2.3, AUX_PWR2.4, AUX_PWR3.3, AUX_PWR3.4, U$8.P$1; no longer AUX_PWR.2, AUX_PWR.5, AUX_PWR1.2, AUX_PWR1.5, AUX_PWR2.2, AUX_PWR2.5, AUX_PWR3.2, AUX_PWR3.5, C6.1, CR1.1, LED5.A, START.RELAY1.86, U$22.P$1, U$23.1
- net 5V: now also AUX_PWR.2, AUX_PWR.5, AUX_PWR1.2, AUX_PWR1.5, AUX_PWR2.2, AUX_PWR2.5, AUX_PWR3.2, AUX_PWR3.5, C2.1; no longer AUX_PWR.3, AUX_PWR.4, AUX_PWR1.3, AUX_PWR1.4, AUX_PWR2.3, AUX_PWR2.4, AUX_PWR3.3, AUX_PWR3.4, U$27.CIRCUIT1
- net GND: no longer AUX_PWR.SH1, AUX_PWR.SH2, AUX_PWR1.SH1, AUX_PWR1.SH2, AUX_PWR2.SH1, AUX_PWR2.SH2, AUX_PWR3.SH1, AUX_PWR3.SH2, C6.2, R12.1, R8.1, U$17.CIRCUIT2, U$22.P$2, U$23.3, U$23.5, U$23.GROUND, U$24.P$2, U$26.CIRCUIT2, U$27.CIRCUIT2
- net VIN: now also JP2.2, U$12.P$1, U$13.OUT
Routing:
- net GND: track 0.00 -> 402.5 mm, vias 0 -> 9
- net 12V: track 0.00 -> 392.0 mm, vias 0 -> 4
- net 5V: track 0.00 -> 157.1 mm, vias 0 -> 4
- net GNDIN: track 0.00 -> 96.7 mm, vias 0 -> 1
- net N$1: track 0.00 -> 57.8 mm
- net VIN_: track 0.00 -> 32.4 mm
- net VIN: track 0.00 -> 30.7 mm, vias 0 -> 1
- net CTRL: track 0.00 -> 28.6 mm
- net N$3: track 0.00 -> 5.21 mm
- net N$6: track 0.00 -> 3.08 mm
- net N$9: track 0.00 -> 2.88 mm
Other:
- board size 100 x 100 mm -> 100 x 80 mm
