File: Milled Version/Aux_Power_Board.sch (EAGLE design)
At the start: 71 parts

Commit message: Made changes to aux power board, created horn board
Parts:
- removed C3: 10uF, SparkFun-Capacitors:1.0UF-0805-25V-10%
- removed C4, C5, C6: 0.1uF, SparkFun-Capacitors:1.0UF-0805-25V-10%
- removed CR1, CR2: MUR420RLG, MUR420RLG - Diode:MUR420RLG
- removed FRAME3, FRAME4: FRAME-LEDGER, SparkFun-Aesthetics:FRAME-LEDGER
- removed JP3: (no value), jumper:JP1E
- removed LED4, LED5, LED6, LED7: (no value), led:LEDCHIP-LED0805
- removed R10, R11, R12, R13: (no value), rcl:R-US_M0805
- removed R4: 100k, SparkFun-Resistors:0.22OHM-0805-1/4W-1%
- removed R5, R8, R9: 8.1MEG, SparkFun-Resistors:0.22OHM-0805-1/4W-1%
- removed R6: 66.67k, SparkFun-Resistors:0.22OHM-0805-1/4W-1%
- removed R7: 233.33k, SparkFun-Resistors:0.22OHM-0805-1/4W-1%
- removed START.RELAY1: VCF4-1000, VCF4-1000:VCF4-1000
- removed U$11: CAP-8MM3.5MM, Eagle Library:CAP-8MM3.5MM
- removed U$16, U$20: FUSEMINI-BLADE, Shell2013:FUSEMINI-BLADE
- removed U$17, U$18, U$21, U$26, U$27: TE770966, Shell2013(1):TE770966
- removed U$19: 5W_RESISTOR, Eagle Library:5W_RESISTOR
- removed U$22, U$24: CAPESK108M025AH4EA, Shell2015:CAPESK108M025AH4EA
- removed U$23: LM2576, Shell2015:LM2576
- removed U$25: M1418-ND, Shell2015:M1418-ND
- removed U$5: LT4365, Eagle Library:LT4365
- removed U$6: SI4946, Eagle Library:SI4946
- C1, C2: value 0.1uF -> (none); device SparkFun-Capacitors:1.0UF-0805-25V-10% -> E-P-099-R2.2:CAP0805
- U$8: value MBR360GOS -> CAPESK107M025AC3AA; device Shell2013:MBR360GOS -> Shell2015:CAPESK107M025AC3AA
Connections:
- net VIN_UNFUSED renamed VIN_
- removed net BATTERY_GND: C3.2, C4.2, C5.2, JP1.1, R1.1, R7.1, START.RELAY1.30, U$11.-, U$12.GNDIN, U$14.G/LOW, U$15.G/LOW, U$21.G/LOW, U$5.GND
- removed net FAULT': R10.1, U$5.FAULT'
- removed net GATE: U$5.GATE, U$6.G1, U$6.G2
- removed net N$10: CR2.2, U$18.V/SIG, U$19.2
- removed net N$11: CR1.2, R11.1, START.RELAY1.85, U$17.V/SIG
- removed net N$12: R13.2, START.RELAY1.87, U$19.1
- removed net N$13: JP3.1, R4.2
- removed net N$14: U$20.IN, U$21.V/SIG
- removed net N$15: U$23.OUTPUT, U$25.P$1, U$8.P$2
- removed net N$16: R8.2, R9.1, U$23.FEEDBACK
- removed net N$17: LED4.C, R10.2
- removed net N$18: LED5.C, R11.2
- removed net N$19: LED6.C, R12.2
- removed net N$2: R4.1, U$5.SHDN'
- removed net N$20: LED7.C, R13.1
- removed net N$4: R5.1, R6.2, U$5.UV
- removed net N$5: R6.1, R7.2, U$5.OV
- removed net N$8: CR2.1, LED7.A, U$16.OUT, U$18.G/LOW
- removed net SERVO_POWER: C2.1, LED6.A, R9.2, U$24.P$1, U$25.P$2, U$26.V/SIG
- removed net SOURCE1: U$6.S1, U$6.S2
- removed net VIN_FUSED: C3.1, C4.1, JP3.2, LED4.A, R5.2, U$13.OUT, U$5.VIN, U$6.D1, U$6.D1_#2
- removed net VIN_PROTECTED: C5.1, JP2.2, U$11.+, U$12.VIN, U$16.IN, U$20.OUT, U$5.VOUT, U$6.D2, U$6.D2_#2
- new net GNDIN: JP1.1, R1.1, U$12.GNDIN, U$14.G/LOW, U$15.G/LOW
- net 12V: now also AUX_PWR.3, AUX_PWR.4, AUX_PWR1.3, AUX_PWR1.4, AUX_PWR2.3, AUX_PWR2.4, AUX_PWR3.3, AUX_PWR3.4, U$8.P$1; no longer AUX_PWR.2, AUX_PWR.5, AUX_PWR1.2, AUX_PWR1.5, AUX_PWR2.2, AUX_PWR2.5, AUX_PWR3.2, AUX_PWR3.5, C6.1, CR1.1, LED5.A, START.RELAY1.86, U$22.P$1, U$23.VIN
- net 5V: now also AUX_PWR.2, AUX_PWR.5, AUX_PWR1.2, AUX_PWR1.5, AUX_PWR2.2, AUX_PWR2.5, AUX_PWR3.2, AUX_PWR3.5, C2.1; no longer AUX_PWR.3, AUX_PWR.4, AUX_PWR1.3, AUX_PWR1.4, AUX_PWR2.3, AUX_PWR2.4, AUX_PWR3.3, AUX_PWR3.4, U$27.V/SIG
- net GND: now also U$8.P$2; no longer AUX_PWR.SH1, AUX_PWR.SH2, AUX_PWR1.SH1, AUX_PWR1.SH2, AUX_PWR2.SH1, AUX_PWR2.SH2, AUX_PWR3.SH1, AUX_PWR3.SH2, C6.2, R12.1, R8.1, U$17.G/LOW, U$22.P$2, U$23.GROUND, U$23.ON/OFF, U$24.P$2, U$26.G/LOW, U$27.G/LOW, U$8.P$1
- net VIN: now also JP2.2, U$12.VIN, U$13.OUT
Other:
- note removed: "1.5 OHM"
- note removed: "1000uF"
- note removed: "220 uF 493-1302-ND"
- note removed: "493-13452-1-ND"
- note removed: "5V Regulator"
- note removed: "Adjustable Servo Regulator"
- note removed: "Battery Input"
- note removed: "Dedicated Horn Fuse"
- note removed: "Filter caps on 12V regulator input"
- note removed: "Filter caps on 12V regulator output"
- note removed: "Flyback Diode"
- note removed: "Horn Button Connector"
- note removed: "Horn Circuit"
- note removed: "Horn Connector"
- note removed: "Output Connectors"
- note removed: "Protection IC Bypass (in case it doesn't work)"
- note removed: "Recom 12V Isolated Regulator"
- note removed: "Under/Over Voltage and Reverse Polarity Protection"
- note removed: "increase pad size later"
- note removed: "review this package later"
