File: V5.0/Horn Board/Horn_Board/Horn_Board.brd (EAGLE design)
At the start: 75 x 75 mm, 21 parts, among them J1 455-1750-1-ND

Commit message: Horn Board almost 100%
Finished horn board, just need to review. Made a few changes to the aux power board, still a work in progress
Parts:
- removed C1, C5: 0.1uF, SparkFun-Capacitors:0805
- removed J1: 455-1750-1-ND, SparkFun-Connectors:1X03
- removed JP3: (no value), jumper:JP1
- removed START.RELAY1: VCF4-1000, VCF4-1000:VCF4-1000
- removed U$5: L4931CD120-TR, Eagle Library:SOIC127P600X175-8N
- removed U$8: CAPESK107M025AC3AA, Shell2015:ESK107M025AC3AA
- added H1, H2, H3, H4: STAND-OFF, SparkFun-Electromechanical:STAND-OFF
- added LED1: (no value), led:CHIP-LED0805
- added R1: (no value), rcl:M0805
- added U$7: 0.250W_RES, Eagle Library:AXIAL-0.3
- U$3: value 10W_RESISTOR -> OMRON_G5LE-1; device Eagle Library:10W_RESISTOR -> Eagle Library:OMRON_G5LE-1
- U$4: value 1W_RESISTOR -> 10W_RESISTOR; device Eagle Library:1W_RESISTOR -> Eagle Library:10W_RESISTOR
- moved U$4 160.8 mm to (50.3, 36.5)
- moved U$17 88.5 mm to (-1.13, 61.4), turned to 270 degrees
- moved LED7 83.1 mm to (25.6, 18.8), turned to 90 degrees
- moved R13 82.0 mm to (19.1, 18.8), turned to 180 degrees
- moved R11 81.6 mm to (19.1, 22.8)
- moved LED5 77.0 mm to (25.6, 22.8), turned to 90 degrees
- moved U$18 72.3 mm to (-1.23, 12.7), turned to 270 degrees
- moved U$1 68.6 mm to (-1.13, 46.8), turned to 270 degrees
- moved U$2 42.5 mm to (2.50, 30.2), turned to 270 degrees
- moved CR2 37.4 mm to (21.0, 7.92)
- moved U$3 25.6 mm to (29.8, 59.1), turned to 270 degrees
- moved U$11 14.8 mm to (20.6, 34.4), turned to 90 degrees
- moved CR1 11.7 mm to (20.2, 42.4)
Connections:
- removed net 12V: CR1.1, LED5.A, START.RELAY1.86, U$5.1
- removed net 12V_REG_IN: J1.3, U$5.8
- removed net BATTERY_GND: START.RELAY1.30
- removed net N$10: CR2.2, U$18.CIRCUIT1, U$3.P$2
- removed net N$11: CR1.2, R11.1, START.RELAY1.85, U$17.CIRCUIT1
- removed net N$12: R13.2, START.RELAY1.87, U$3.P$1
- removed net N$2: U$4.P$2
- new net COIL_POWER: CR1.1, LED5.A, U$3.5, U$7.P$1
- new net HORN-: CR2.2, R13.2, U$18.CIRCUIT2, U$4.P$2
- new net HORN_BUTTON: CR1.2, R11.1, U$17.CIRCUIT1, U$3.2
- new net N$5: LED1.C, R1.2
- net GND: now also R1.1, U$3.1; no longer C5.2, U$5.2, U$5.3, U$5.5, U$5.6, U$5.7, U$8.P$2
- net N$1: now also U$3.3; no longer J1.1
- net VIN_FUSED: now also LED1.A, U$18.CIRCUIT1, U$7.P$2; no longer C5.1, J1.2, U$18.CIRCUIT2
Routing:
- net VIN_FUSED: track 0.00 -> 91.8 mm
- net HORN_BUTTON: track 0.00 -> 76.8 mm, vias 0 -> 2
- net GND: track 0.00 -> 62.7 mm, vias 0 -> 1
- net COIL_POWER: track 0.00 -> 56.3 mm, vias 0 -> 1
- net HORN-: track 0.00 -> 51.5 mm, vias 0 -> 1
- net VIN_UNFUSED: track 0.00 -> 26.5 mm
- net N$1: track 0.00 -> 24.2 mm
- net N$5: track 0.00 -> 4.50 mm
- net N$20: track 0.00 -> 4.50 mm
- net N$18: track 0.00 -> 4.50 mm
Other:
- board size 75 x 75 mm -> 60 x 75 mm
- board text added: "Button"
- board text added: "Horn"
- board text added: "Horn Out"
- board text added: "Power"
- board text added: "Relay Coil"
- board text added: "VIN"
