File: V5.0/Horn Board/Horn_Board/Horn_Board.sch (EAGLE design)
At the start: 71 parts

Commit message: Made changes to aux power board, created horn board
Parts:
- removed AUX_PWR, AUX_PWR1, AUX_PWR2, AUX_PWR3: 5555140-6, 5555140-6 RJ11:5555140-6
- removed C2, C4, C6: 0.1uF, SparkFun-Capacitors:1.0UF-0805-25V-10%
- removed C3: 10uF, SparkFun-Capacitors:1.0UF-0805-25V-10%
- removed FRAME2, FRAME3, FRAME4: FRAME-LEDGER, SparkFun-Aesthetics:FRAME-LEDGER
- removed H1, H2, H3, H4: STAND-OFF, SparkFun-Electromechanical:STAND-OFF
- removed JP1, JP2: (no value), jumper:JP1E
- removed LED1, LED2, LED3, LED4, LED6: (no value), led:LEDCHIP-LED0805
- removed R1, R10, R12, R2, R3: (no value), rcl:R-US_M0805
- removed R4: 100k, SparkFun-Resistors:0.22OHM-0805-1/4W-1%
- removed R5, R8, R9: 8.1MEG, SparkFun-Resistors:0.22OHM-0805-1/4W-1%
- removed R6: 66.67k, SparkFun-Resistors:0.22OHM-0805-1/4W-1%
- removed R7: 233.33k, SparkFun-Resistors:0.22OHM-0805-1/4W-1%
- removed U$10, U$25: M1418-ND, Shell2015:M1418-ND
- removed U$12: RPA60-2412SFW_P, RPA60-2412SFW_P:RPA60-2412SFW_P
- removed U$13, U$16, U$20: FUSEMINI-BLADE, Shell2013:FUSEMINI-BLADE
- removed U$14, U$15, U$21, U$26, U$27: TE770966, Shell2013(1):TE770966
- removed U$19: 5W_RESISTOR, Eagle Library:5W_RESISTOR
- removed U$22, U$24, U$9: CAPESK108M025AH4EA, Shell2015:CAPESK108M025AH4EA
- removed U$23, U$7: LM2576, Shell2015:LM2576
- removed U$6: SI4946, Eagle Library:SI4946
- added J1: 455-1750-1-ND, SparkFun-Connectors:CONN_03
- U$2: value TE770966 -> FUSEMINI-BLADE; device Shell2013(1):TE770966 -> Shell2013:FUSEMINI-BLADE
- U$3: value TE770966 -> 10W_RESISTOR; device Shell2013(1):TE770966 -> Eagle Library:10W_RESISTOR
- U$4: value MBR360GOS -> 1W_RESISTOR; device Shell2013:MBR360GOS -> Eagle Library:1W_RESISTOR
- U$5: value LT4365 -> L4931CD120-TR; device Eagle Library:LT4365 -> Eagle Library:L4931CD120-TR
- U$8: value MBR360GOS -> CAPESK107M025AC3AA; device Shell2013:MBR360GOS -> Shell2015:CAPESK107M025AC3AA
Connections:
- removed net 5V: AUX_PWR.3, AUX_PWR.4, AUX_PWR1.3, AUX_PWR1.4, AUX_PWR2.3, AUX_PWR2.4, AUX_PWR3.3, AUX_PWR3.4, C1.1, LED1.A, U$10.P$2, U$27.V/SIG, U$3.V/SIG, U$7.FEEDBACK, U$9.P$1
- removed net CTRL: JP2.1, U$12.CRTL
- removed net FAULT': R10.1, U$5.FAULT'
- removed net GATE: U$5.GATE, U$6.G1, U$6.G2
- removed net N$13: JP3.1, R4.2
- removed net N$14: U$20.IN, U$21.V/SIG
- removed net N$15: U$23.OUTPUT, U$25.P$1, U$8.P$2
- removed net N$16: R8.2, R9.1, U$23.FEEDBACK
- removed net N$17: LED4.C, R10.2
- removed net N$19: LED6.C, R12.2
- removed net N$3: LED3.C, R1.2
- removed net N$4: R5.1, R6.2, U$5.UV
- removed net N$5: R6.1, R7.2, U$5.OV
- removed net N$6: LED2.C, R2.2
- removed net N$7: U$12.TRIM
- removed net N$8: CR2.1, LED7.A, U$16.OUT, U$18.G/LOW
- removed net N$9: LED1.C, R3.2
- removed net SERVO_POWER: C2.1, LED6.A, R9.2, U$24.P$1, U$25.P$2, U$26.V/SIG
- removed net SOURCE1: U$6.S1, U$6.S2
- removed net VIN: LED3.A
- removed net VIN_PROTECTED: C5.1, JP2.2, U$11.+, U$12.VIN, U$16.IN, U$20.OUT, U$5.VOUT, U$6.D2, U$6.D2_#2
- new net 12V_REG_IN: J1.3, U$5.VIN
- net 12V: now also U$5.VOUT; no longer AUX_PWR.2, AUX_PWR.5, AUX_PWR1.2, AUX_PWR1.5, AUX_PWR2.2, AUX_PWR2.5, AUX_PWR3.2, AUX_PWR3.5, C6.1, LED2.A, U$1.V/SIG, U$12.VOUT, U$2.V/SIG, U$22.P$1, U$23.VIN, U$7.VIN
- net BATTERY_GND: no longer C3.2, C4.2, C5.2, JP1.1, R1.1, R7.1, U$11.-, U$12.GNDIN, U$14.G/LOW, U$15.G/LOW, U$21.G/LOW, U$5.GND
- net GND: now also C5.2, U$11.-, U$5.GND1, U$5.GND2, U$5.GND3, U$5.GND4, U$5.INHIBIT, U$8.P$2; no longer AUX_PWR.1, AUX_PWR.6, AUX_PWR.SH1, AUX_PWR.SH2, AUX_PWR1.1, AUX_PWR1.6, AUX_PWR1.SH1, AUX_PWR1.SH2, AUX_PWR2.1, AUX_PWR2.6, AUX_PWR2.SH1, AUX_PWR2.SH2, AUX_PWR3.1, AUX_PWR3.6, AUX_PWR3.SH1, AUX_PWR3.SH2, C1.2, C2.2, C6.2, JP1.2, R12.1, R2.1, R3.1, R8.1, U$12.GNDOUT, U$2.G/LOW, U$22.P$2, U$23.GROUND, U$23.ON/OFF, U$24.P$2, U$26.G/LOW, U$27.G/LOW, U$3.G/LOW, U$4.P$1, U$7.GROUND, U$7.ON/OFF, U$8.P$1, U$9.P$2
- net N$1: now also J1.1, U$4.1; no longer U$10.P$1, U$4.P$2, U$7.OUTPUT
- net N$10: now also U$3.2; no longer U$19.2
- net N$12: now also U$3.1; no longer U$19.1
- net N$2: now also U$4.2; no longer R4.1, U$5.SHDN'
- net VIN_FUSED: now also C5.1, CR2.1, J1.2, LED7.A, U$11.+, U$18.G/LOW, U$2.OUT; no longer C3.1, C4.1, JP3.2, LED4.A, R5.2, U$13.OUT, U$5.VIN, U$6.D1, U$6.D1_#2
- net VIN_UNFUSED: now also U$1.V/SIG, U$2.IN; no longer U$13.IN, U$14.V/SIG, U$15.V/SIG
Other:
- note removed: "1000uF"
- note removed: "493-13452-1-ND"
- note removed: "5V Regulator"
- note removed: "Adjustable Servo Regulator"
- note removed: "Aux Power"
- note removed: "Battery Input"
- note removed: "Dedicated Horn Fuse"
- note removed: "Filter caps on 12V regulator input"
- note removed: "Filter caps on 12V regulator output"
- note removed: "Horn Circuit"
- note removed: "Output Connectors"
- note removed: "Protection IC Bypass (in case it doesn't work)"
- note removed: "Recom 12V Isolated Regulator"
- note removed: "Under/Over Voltage and Reverse Polarity Protection"
- note removed: "increase pad size later"
- note removed: "review this package later"

Commit message: Horn Board almost 100%
Finished horn board, just need to review. Made a few changes to the aux power board, still a work in progress
Parts:
- removed C1, C5: 0.1uF, SparkFun-Capacitors:1.0UF-0805-25V-10%
- removed J1: 455-1750-1-ND, SparkFun-Connectors:CONN_03
- removed JP3: (no value), jumper:JP1E
- removed START.RELAY1: VCF4-1000, VCF4-1000:VCF4-1000
- removed U$5: L4931CD120-TR, Eagle Library:L4931CD120-TR
- removed U$8: CAPESK107M025AC3AA, Shell2015:CAPESK107M025AC3AA
- added H1, H2, H3, H4: STAND-OFF, SparkFun-Electromechanical:STAND-OFF
- added LED1: (no value), led:LEDCHIP-LED0805
- added R1: (no value), rcl:R-US_M0805
- added U$7: 0.250W_RES, Eagle Library:0.250W_RES
- U$3: value 10W_RESISTOR -> OMRON_G5LE-1; device Eagle Library:10W_RESISTOR -> Eagle Library:OMRON_G5LE-1
- U$4: value 1W_RESISTOR -> 10W_RESISTOR; device Eagle Library:1W_RESISTOR -> Eagle Library:10W_RESISTOR
Connections:
- removed net 12V: CR1.1, LED5.A, START.RELAY1.86, U$5.VOUT
- removed net 12V_REG_IN: J1.3, U$5.VIN
- removed net BATTERY_GND: START.RELAY1.30
- removed net N$10: CR2.2, U$18.V/SIG, U$3.2
- removed net N$11: CR1.2, R11.1, START.RELAY1.85, U$17.V/SIG
- removed net N$12: R13.2, START.RELAY1.87, U$3.1
- removed net N$2: U$4.2
- new net COIL_POWER: CR1.1, LED5.A, U$3.86, U$7.1
- new net HORN-: CR2.2, R13.2, U$18.G/LOW, U$4.2
- new net HORN_BUTTON: CR1.2, R11.1, U$17.V/SIG, U$3.85
- new net N$5: LED1.C, R1.2
- net GND: now also R1.1, U$3.30; no longer C5.2, U$5.GND1, U$5.GND2, U$5.GND3, U$5.GND4, U$5.INHIBIT, U$8.P$2
- net N$1: now also U$3.87; no longer J1.1
- net VIN_FUSED: now also LED1.A, U$18.V/SIG, U$7.2; no longer C5.1, J1.2, U$18.G/LOW
Other:
- note added: "150 Ohm, S150CACT-ND"
- note added: "750 ohm, P750ADDKR-ND"
- note added: "Horn Indication"
- note added: "Horn Relay Indication"
- note added: "Power Indication"
- note added: "Z3672-ND"
- moved on the sheet: CR1, CR2, LED5, LED7, R11, R13, U$11, U$4
