File: V5.0/Aux_Power_Board.brd (EAGLE design)
At the start: 100 x 100 mm, 71 parts

Commit message: Horn Board almost 100%
Finished horn board, just need to review. Made a few changes to the aux power board, still a work in progress
Parts:
- removed CR1, CR2: MUR420RLG, MUR420RLG - Diode:DO-201AD
- removed FRAME3: FRAME-LEDGER, SparkFun-Aesthetics:CREATIVE_COMMONS
- removed LED5, LED7: (no value), led:CHIP-LED0805
- removed R11, R13: (no value), rcl:M0805
- removed START.RELAY1: VCF4-1000, VCF4-1000:VCF4-1000
- removed U$15, U$17, U$18: TE770966, Shell2013(1):2X1-MATE-N-LOCK
- removed U$16: FUSEMINI-BLADE, Shell2013:MINI-BLADE-FUSE
- removed U$19: 5W_RESISTOR, Eagle Library:5W_RESISTOR
- moved U$8 316.7 mm to (46.8, 38.7)
- moved U$22 294.2 mm to (65.2, 28.7)
- moved U$24 273.5 mm to (86.8, 17.6)
- moved LED6 257.9 mm to (103.0, -33.8)
- moved R12 229.0 mm to (128.8, -37.8)
- moved U$11 214.7 mm to (80.0, 37.4)
- moved R10 190.5 mm to (158.0, -19.0)
- moved C1 190.5 mm to (160.9, 87.0)
- moved C2 190.5 mm to (181.1, 1.20)
- moved C6 190.5 mm to (160.9, 99.8)
- moved FRAME4 190.5 mm to (176.9, -34.9)
- moved LED4 190.5 mm to (159.1, -25.4)
- moved R8 190.5 mm to (161.1, -13.9)
- moved R9 190.5 mm to (157.6, -13.9)
- moved JP3 190.5 mm to (170.3, 121.8)
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Connections:
- removed net N$10: CR2.2, U$18.CIRCUIT1, U$19.P$2
- removed net N$11: CR1.2, R11.1, START.RELAY1.85, U$17.CIRCUIT1
- removed net N$12: R13.2, START.RELAY1.87, U$19.P$1
- removed net N$18: LED5.C, R11.2
- removed net N$20: LED7.C, R13.1
- removed net N$8: CR2.1, LED7.A, U$16.OUT, U$18.CIRCUIT2
- net 12V: no longer CR1.1, LED5.A, START.RELAY1.86
- net BATTERY_GND: no longer START.RELAY1.30, U$15.CIRCUIT2
- net GND: no longer U$17.CIRCUIT2
- net VIN_PROTECTED: no longer U$16.IN
- net VIN_UNFUSED: no longer U$15.CIRCUIT1

Commit message: More changes
Parts:
- added U$15: TE770966, Shell2013(1):2X1-MATE-N-LOCK
- R8: value 8.1MEG -> 1k
- R9: value 8.1MEG -> 3.9k
- moved U$1 101.8 mm to (101.5, 32.1), turned to 90 degrees
- moved C5 93.9 mm to (40.1, 28.0), flipped to the bottom, turned to 90 degrees
- moved C4 74.1 mm to (26.4, 37.1), flipped to the bottom, turned to 90 degrees
- moved C3 71.5 mm to (23.6, 37.1), flipped to the bottom, turned to 90 degrees
- moved U$23 49.4 mm to (56.4, 52.9)
- moved U$5 41.4 mm to (33.4, 47.0), flipped to the bottom, turned to 180 degrees
- moved U$25 38.9 mm to (57.1, 40.6), flipped to the bottom, turned to 270 degrees
- moved U$11 34.2 mm to (48.5, 24.2), turned to 90 degrees
- moved U$24 31.3 mm to (66.4, 41.4)
- moved U$6 25.1 mm to (29.9, 31.7), flipped to the bottom
- moved U$9 15.1 mm to (85.8, 43.4)
- moved U$3 14.2 mm to (76.2, -1.20)
- moved U$27 10.7 mm to (60.6, -1.20)
- moved U$10 8.79 mm to (74.4, 65.5), flipped to the bottom, turned to 180 degrees
- moved U$26 8.37 mm to (44.2, -1.20)
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Connections:
- net GND: now also U$15.CIRCUIT2
- net VIN_PROTECTED: now also U$15.CIRCUIT1
Routing:
- net VIN_FUSED: track 0.00 -> 42.9 mm
- net VIN_PROTECTED: track 0.00 -> 29.6 mm
- net VIN_UNFUSED: track 0.00 -> 15.7 mm
- net BATTERY_GND: track 0.00 -> 11.2 mm
