File: V5.0/Aux_Power_Board.sch (EAGLE design)
At the start: 71 parts

Commit message: Horn Board almost 100%
Finished horn board, just need to review. Made a few changes to the aux power board, still a work in progress
Parts:
- removed CR1, CR2: MUR420RLG, MUR420RLG - Diode:MUR420RLG
- removed FRAME3: FRAME-LEDGER, SparkFun-Aesthetics:FRAME-LEDGER
- removed LED5, LED7: (no value), led:LEDCHIP-LED0805
- removed R11, R13: (no value), rcl:R-US_M0805
- removed START.RELAY1: VCF4-1000, VCF4-1000:VCF4-1000
- removed U$15, U$17, U$18: TE770966, Shell2013(1):TE770966
- removed U$16: FUSEMINI-BLADE, Shell2013:FUSEMINI-BLADE
- removed U$19: 5W_RESISTOR, Eagle Library:5W_RESISTOR
Connections:
- removed net N$10: CR2.2, U$18.V/SIG, U$19.2
- removed net N$11: CR1.2, R11.1, START.RELAY1.85, U$17.V/SIG
- removed net N$12: R13.2, START.RELAY1.87, U$19.1
- removed net N$18: LED5.C, R11.2
- removed net N$20: LED7.C, R13.1
- removed net N$8: CR2.1, LED7.A, U$16.OUT, U$18.G/LOW
- net 12V: no longer CR1.1, LED5.A, START.RELAY1.86
- net BATTERY_GND: no longer START.RELAY1.30, U$15.G/LOW
- net GND: no longer U$17.G/LOW
- net VIN_PROTECTED: no longer U$16.IN
- net VIN_UNFUSED: no longer U$15.V/SIG
Other:
- note removed: "1.5 OHM"
- note removed: "Dedicated Horn Fuse"
- note removed: "Flyback Diode"
- note removed: "Horn Button Connector"
- note removed: "Horn Circuit"
- note removed: "Horn Connector"

Commit message: More changes
Parts:
- added U$15: TE770966, Shell2013(1):TE770966
- R8: value 8.1MEG -> 1k
- R9: value 8.1MEG -> 3.9k
Connections:
- net GND: now also U$15.G/LOW
- net VIN_PROTECTED: now also U$15.V/SIG
Other:
- note added: "12V Power"
- note added: "150uH or 220uH"
- note added: "220uH"
- note added: "5V Power"
- note added: "Battery Power"
- note added: "Fault"
- note added: "Horn Power"
- note added: "Servo Power"
- moved on the sheet: LED1, LED3, LED4, LED6, R1, R10, R12, R3
Changed lines of the file:
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@@
 <part name="U$25" library="Shell2015" deviceset="M1418-ND" device=""/>
 <part name="C2" library="SparkFun-Capacitors" deviceset="1.0UF" device="-0805-25V-10%" value="0.1uF"/>
-<part name="R8" library="SparkFun-Resistors" deviceset="0.22OHM" device="-0805-1/4W-1%" value="8.1MEG"/>
-<part name="R9" library="SparkFun-Resistors" deviceset="0.22OHM" device="-0805-1/4W-1%" value="8.1MEG"/>
+<part name="R8" library="SparkFun-Resistors" deviceset="0.22OHM" device="-0805-1/4W-1%" value="1k"/>
+<part name="R9" library="SparkFun-Resistors" deviceset="0.22OHM" device="-0805-1/4W-1%" value="3.9k"/>
 <part name="LED4" library="led" library_urn="urn:adsk.eagle:library:259" deviceset="LED" device="CHIP-LED0805" package3d_urn="urn:adsk.eagle:package:15818/2"/>
 <part name="R10" library="rcl" library_urn="urn:adsk.eagle:library:334" deviceset="R-US_" device="M0805" package3d_urn="urn:adsk.eagle:package:23556/1"/>
@@
 <part name="R12" library="rcl" library_urn="urn:adsk.eagle:library:334" deviceset="R-US_" device="M0805" package3d_urn="urn:adsk.eagle:package:23556/1"/>
 <part name="U$27" library="Shell2013(1)" deviceset="TE770966" device=""/>
+<part name="U$15" library="Shell2013(1)" deviceset="TE770966" device=""/>
 </parts>
 <sheets>
@@
 <text x="109.22" y="83.82" size="1.778" layer="94">1000uF</text>
 <text x="38.1" y="129.54" size="3.81" layer="94">Adjustable Servo Regulator</text>
+<text x="208.28" y="236.22" size="1.778" layer="94">Fault</text>
+<text x="251.46" y="236.22" size="1.778" layer="94">Battery Power</text>
+<text x="284.48" y="236.22" size="1.778" layer="94">12V Power</text>
+<text x="325.12" y="236.22" size="1.778" layer="94">5V Power</text>
+<text x="373.38" y="236.22" size="1.778" layer="94">Servo Power</text>
+<text x="101.6" y="91.44" size="1.778" layer="94">220uH</text>
+<text x="86.36" y="220.98" size="1.778" layer="94">150uH or 220uH</text>
 </plain>
 <instances>
@@
 <instance part="U$9" gate="G$1" x="111.76" y="213.36" rot="R270"/>
 <instance part="U$10" gate="G$1" x="91.44" y="226.06"/>
-<instance part="LED1" gate="G$1" x="312.42" y="220.98"/>
+<instance part="LED1" gate="G$1" x="325.12" y="220.98"/>
 <instance part="LED2" gate="G$1" x="287.02" y="220.98"/>
-<instance part="LED3" gate="G$1" x="259.08" y="220.98"/>
-<instance part="R1" gate="G$1" x="259.08" y="203.2" rot="R90"/>
+<instance part="LED3" gate="G$1" x="251.46" y="220.98"/>
+<instance part="R1" gate="G$1" x="251.46" y="203.2" rot="R90"/>
 <instance part="R2" gate="G$1" x="287.02" y="203.2" rot="R90"/>
-<instance part="R3" gate="G$1" x="312.42" y="203.2" rot="R90"/>
+<instance part="R3" gate="G$1" x="325.12" y="203.2" rot="R90"/>
 <instance part="FRAME1" gate="G$1" x="0" y="0"/>
 <instance part="FRAME1" gate="G$2" x="330.2" y="0"/>
@@
 <instance part="R8" gate="G$1" x="60.96" y="93.98" rot="R180"/>
 <instance part="R9" gate="G$1" x="45.72" y="93.98" rot="R180"/>
-<instance part="LED4" gate="G$1" x="231.14" y="220.98"/>
-<instance part="R10" gate="G$1" x="231.14" y="203.2" rot="R90"/>
-<instance part="LED6" gate="G$1" x="337.82" y="220.98"/>
-<instance part="R12" gate="G$1" x="337.82" y="203.2" rot="R90"/>
+<instance part="LED4" gate="G$1" x="208.28" y="220.98"/>
+<instance part="R10" gate="G$1" x="208.28" y="203.2" rot="R90"/>
+<instance part="LED6" gate="G$1" x="373.38" y="220.98"/>
+<instance part="R12" gate="G$1" x="373.38" y="203.2" rot="R90"/>
 </instances>
 <busses>
@@
 <segment>
 <pinref part="R3" gate="G$1" pin="1"/>
-<wire x1="312.42" y1="193.04" x2="312.42" y2="198.12" width="0.1524" layer="91"/>
-<label x="317.754" y="192.278" size="1.778" layer="95" rot="R180"/>
+<wire x1="325.12" y1="193.04" x2="325.12" y2="198.12" width="0.1524" layer="91"/>
+<label x="330.454" y="192.278" size="1.778" layer="95" rot="R180"/>
 </segment>
 <segment>
@@
 <segment>
 <pinref part="R12" gate="G$1" pin="1"/>
-<wire x1="337.82" y1="193.04" x2="337.82" y2="198.12" width="0.1524" layer="91"/>
-<label x="343.154" y="192.278" size="1.778" layer="95" rot="R180"/>
+<wire x1="373.38" y1="193.04" x2="373.38" y2="198.12" width="0.1524" layer="91"/>
+<label x="378.714" y="192.278" size="1.778" layer="95" rot="R180"/>
 </segment>
 </net>
@@
 <segment>
 <pinref part="LED1" gate="G$1" pin="A"/>
-<wire x1="312.42" y1="223.52" x2="312.42" y2="228.6" width="0.1524" layer="91"/>
-<label x="312.42" y="228.6" size="1.778" layer="95"/>
+<wire x1="325.12" y1="223.52" x2="325.12" y2="228.6" width="0.1524" layer="91"/>
+<label x="325.12" y="228.6" size="1.778" layer="95"/>
 </segment>
 <segment>
@@
 <segment>
 <pinref part="R1" gate="G$1" pin="1"/>
-<wire x1="259.08" y1="198.12" x2="259.08" y2="193.04" width="0.1524" layer="91"/>
-<label x="259.08" y="190.5" size="1.778" layer="95"/>
+<wire x1="251.46" y1="198.12" x2="251.46" y2="193.04" width="0.1524" layer="91"/>
+<label x="251.46" y="190.5" size="1.778" layer="95"/>
 </segment>
 </net>
@@
 <pinref part="R1" gate="G$1" pin="2"/>
 <pinref part="LED3" gate="G$1" pin="C"/>
-<wire x1="259.08" y1="208.28" x2="259.08" y2="215.9" width="0.1524" layer="91"/>
+<wire x1="251.46" y1="208.28" x2="251.46" y2="215.9" width="0.1524" layer="91"/>
 </segment>
 </net>
@@
 <segment>
 <pinref part="LED3" gate="G$1" pin="A"/>
-<wire x1="259.08" y1="223.52" x2="259.08" y2="228.6" width="0.1524" layer="91"/>
-<label x="259.08" y="228.6" size="1.778" layer="95"/>
+<wire x1="251.46" y1="223.52" x2="251.46" y2="228.6" width="0.1524" layer="91"/>
+<label x="251.46" y="228.6" size="1.778" layer="95"/>
 </segment>
 </net>
@@
 <pinref part="R3" gate="G$1" pin="2"/>
 <pinref part="LED1" gate="G$1" pin="C"/>
-<wire x1="312.42" y1="208.28" x2="312.42" y2="215.9" width="0.1524" layer="91"/>
+<wire x1="325.12" y1="208.28" x2="325.12" y2="215.9" width="0.1524" layer="91"/>
 </segment>
 </net>
@@
 <segment>
 <pinref part="LED6" gate="G$1" pin="A"/>
-<wire x1="337.82" y1="223.52" x2="337.82" y2="228.6" width="0.1524" layer="91"/>
-<label x="337.82" y="228.6" size="1.778" layer="95"/>
+<wire x1="373.38" y1="223.52" x2="373.38" y2="228.6" width="0.1524" layer="91"/>
+<label x="373.38" y="228.6" size="1.778" layer="95"/>
 </segment>
 </net>
@@
 <pinref part="R10" gate="G$1" pin="2"/>
 <pinref part="LED4" gate="G$1" pin="C"/>
-<wire x1="231.14" y1="208.28" x2="231.14" y2="215.9" width="0.1524" layer="91"/>
+<wire x1="208.28" y1="208.28" x2="208.28" y2="215.9" width="0.1524" layer="91"/>
 </segment>
 </net>
@@
 <segment>
 <pinref part="LED4" gate="G$1" pin="A"/>
-<wire x1="231.14" y1="223.52" x2="231.14" y2="228.6" width="0.1524" layer="91"/>
-<label x="231.14" y="228.6" size="1.778" layer="95"/>
+<wire x1="208.28" y1="223.52" x2="208.28" y2="228.6" width="0.1524" layer="91"/>
+<label x="208.28" y="228.6" size="1.778" layer="95"/>
 </segment>
 </net>
@@
 <segment>
 <pinref part="R10" gate="G$1" pin="1"/>
-<wire x1="231.14" y1="198.12" x2="231.14" y2="193.04" width="0.1524" layer="91"/>
-<label x="231.14" y="190.5" size="1.778" layer="95"/>
+<wire x1="208.28" y1="198.12" x2="208.28" y2="193.04" width="0.1524" layer="91"/>
+<label x="208.28" y="190.5" size="1.778" layer="95"/>
 </segment>
 </net>
@@
 <pinref part="R12" gate="G$1" pin="2"/>
 <pinref part="LED6" gate="G$1" pin="C"/>
-<wire x1="337.82" y1="208.28" x2="337.82" y2="215.9" width="0.1524" layer="91"/>
+<wire x1="373.38" y1="208.28" x2="373.38" y2="215.9" width="0.1524" layer="91"/>
 </segment>
 </net>
@@
 <text x="58.42" y="152.4" size="1.778" layer="94">Aux Power</text>
 <text x="132.08" y="152.4" size="1.778" layer="94">Aux Power</text>
+<text x="203.2" y="160.02" size="1.778" layer="94">Horn Power</text>
 </plain>
 <instances>
@@
 <instance part="U$2" gate="G$1" x="228.6" y="215.9" rot="R270"/>
 <instance part="U$3" gate="G$1" x="254" y="215.9" rot="R270"/>
-<instance part="H1" gate="G$1" x="309.88" y="218.44"/>
-<instance part="H2" gate="G$1" x="325.12" y="220.98"/>
-<instance part="H3" gate="G$1" x="312.42" y="205.74"/>
-<instance part="H4" gate="G$1" x="330.2" y="208.28"/>
+<instance part="H1" gate="G$1" x="406.4" y="269.24"/>
+<instance part="H2" gate="G$1" x="419.1" y="269.24"/>
+<instance part="H3" gate="G$1" x="406.4" y="256.54"/>
+<instance part="H4" gate="G$1" x="419.1" y="256.54"/>
 <instance part="U$26" gate="G$1" x="203.2" y="187.96" rot="R270"/>
 <instance part="U$27" gate="G$1" x="254" y="187.96" rot="R270"/>
+<instance part="U$15" gate="G$1" x="203.2" y="149.86" rot="R270"/>
 </instances>
 <busses>
@@
 <label x="264.16" y="185.42" size="1.778" layer="95"/>
 </segment>
+<segment>
+<pinref part="U$15" gate="G$1" pin="G/LOW"/>
+<wire x1="210.82" y1="147.32" x2="213.36" y2="147.32" width="0.1524" layer="91"/>
+<label x="213.36" y="147.32" size="1.778" layer="95"/>
+</segment>
 </net>
 <net name="12V" class="0">
@@
 </segment>
 </net>
+<net name="VIN_PROTECTED" class="0">
+<segment>
+<pinref part="U$15" gate="G$1" pin="V/SIG"/>
+<wire x1="210.82" y1="152.4" x2="213.36" y2="152.4" width="0.1524" layer="91"/>
+<label x="213.36" y="152.4" size="1.778" layer="95"/>
+</segment>
+</net>
